File: Isolater.kicad_sch (KiCad schematic)
At the start: 15 parts, among them J29 DE9_Receptacle, J30 Conn_01x04, J32 Conn_01x04, U1 UCC12040DVE, U2 L7805, U3 ISO1050DUB

Commit message: more layout and memes
Parts:
- C1: value C_Small -> 1u; LibRef (none) -> CL10A105KA8NNNC; SKU (none) -> CL10A105KA8NNNC; Supplier (none) -> Digikey
- C17, C18: LibRef (none) -> CL10B104KB8NNNC; SKU (none) -> CL10B104KB8NNNC; Supplier (none) -> Digikey
- C2: value C_Small -> 100n; LibRef (none) -> CL10B104KB8NNNC; SKU (none) -> CL10B104KB8NNNC; Supplier (none) -> Digikey
- C3: LibRef (none) -> CL10A106MP8NNNC; SKU (none) -> CL10A106MP8NNNC; Supplier (none) -> Digikey
- D1: value D_Schottky -> SSB43L; LibRef (none) -> SSB43L-M3/52T; SKU (none) -> SSB43L-M3/52T; Supplier (none) -> Digikey
- D7: value D_TVS_Dual_AAC -> ESDCAN24-2BLY; SKU (none) -> ESDCAN24-2BLY; Supplier (none) -> Digikey
- J29: value DE9_Receptacle -> Norcomp 172-009-243R021; SKU (none) -> 172-009-243R021; Supplier (none) -> Digikey
- J30, J32: value Conn_01x04 -> Pin Socket 0.1" 01x04; now left out of the parts list
- U1: SKU (none) -> UCC12040DVE; Supplier (none) -> Digikey
- U2: value L7805 -> L7805CDT; LibRef (none) -> L7805CDT-TR; SKU (none) -> L7805CDT-TR; Supplier (none) -> Digikey
- U3: SKU (none) -> ISO1050DUB; Supplier (none) -> Digikey

Commit message: removed slots
Other:
- note removed: "TODO: Figure out passives for this"
Changed lines of the file:
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@@
     (effects (font (size 1.27 1.27)) (justify left bottom))
-  )
-  (text "TODO: Figure out passives for this\n" (at 73.66 77.47 0)
-    (effects (font (size 3 3) (thickness 0.8) bold (color 255 4 17 1)) (justify left bottom))
   )
   (label "GLV-" (at 127 146.05 0) (fields_autoplaced)
