File: cell-tap-connector-pcb.kicad_pcb (KiCad board)
At the start: 4 copper layers, 300.9 x 61.1 mm, 133 parts, among them J1 Conn_01x02, J10 Conn_01x02, J11 Conn_01x02, J12 Conn_01x02, J13 Conn_01x01, J14 Conn_01x01, J15 Conn_01x01, J16 Conn_01x01, J17 Conn_01x01, J18 Conn_01x01, J19 Conn_01x01, J2 Conn_01x02, J20 Conn_01x01, J21 Conn_01x01, J22 Conn_01x01, J23 Conn_01x01, J24 Conn_01x01, J25 Conn_01x01, J26 Conn_01x04, J27 Conn_01x04, J28 TC2030, J29 DE9_Receptacle, J3 Conn_01x02, J30 Conn_01x04, J31 DA15_Receptacle, J32 Conn_01x04, J4 Conn_01x02, J5 Conn_01x02, J6 Conn_01x02, J7 Conn_01x02, J8 Conn_01x02, J9 Conn_01x02, U1 STM32F103R8Tx, U2 UCC12040DVE, U3 L7805, U4 ISO1050DUB, Y1 8MHz

Commit message: more layout and memes
Parts:
- removed mouse-bite-3mm-slot (x3): VAL**, Panelization:mouse-bite-3mm-slot
- added G***: LOGO, art:stickbug, B.Cu at (93.3, 53.4)
- added G***: LOGO, art:pretzel, B.Cu at (132.5, 46.9)
- C27: value C_Small -> 1u
- C28: value C_Small -> 100n
- D10, D11, D12, D13, D14, D15, D17, D3, D5, D6, D7, D8, D9: value RED -> RED 0603
- D18: value D_Schottky -> SSB43L
- D19: value D_TVS_Dual_AAC -> ESDCAN24-2BLY
- F1, F10, F11, F12, F13, F2, F3, F4, F5, F6, F7, F8, F9: value Fuse -> 2A 63VDC 1206
- J1, J10, J11, J12, J2, J3, J4, J5, J6, J7, J8, J9: value Conn_01x02 -> JST S2B-PH-SM4-TB
- J13, J14, J15, J16, J17, J18, J19, J20, J21, J22, J23, J24, J25: value Conn_01x01 -> Mounting Hole M5
- J26, J27: value Conn_01x04 -> Pin Header 0.1" 01x04
- J29: value DE9_Receptacle -> Norcomp 172-009-243R021
- J30, J32: value Conn_01x04 -> Pin Socket 0.1" 01x04
- J31: value DA15_Receptacle -> 172-015-243R021
- TH1, TH3, TH4: value 10k NTC -> 10k NTC ERT-J1VR103J
- U1: value STM32F103R8Tx -> STM32F103R8T6
- U3: value L7805 -> L7805CDT
- Y1: value 8MHz -> 8MHz 20pF
Connections:
- net /Isolater/3v3@HV renamed /Isolator/3v3@HV
- net /Isolater/5V0@GLV renamed /Isolator/5V0@GLV
- net /Isolater/CANH renamed /Isolator/CANH
- net /Isolater/CANL renamed /Isolator/CANL
- net /Isolater/CANRX renamed /Isolator/CANRX
- net /Isolater/CANTX renamed /Isolator/CANTX
- net /Isolater/GLV+ renamed /Isolator/GLV+
- net /Isolater/GLV- renamed /Isolator/GLV-
- net /Isolater/GND@HV renamed /Isolator/GND@HV
Other:
- board text added: "+ 10 8 6 4 2 -"
- board text added: "+ H + H"
- board text added: "- L - L"
- board text added: "11 9 7 5 3 1"
- board text added: "if you are reading this text, this segment is assembled incorrectly."
- board text added: "you just lost the game"
- board text removed: "if you are reading this text, this segment is not assembled correctly"

Commit message: removed slots
Parts:
- added mouse-bite-3mm-slot: VAL**, Panelization:mouse-bite-3mm-slot, F.Cu at (301.0, 59.0)
- added mouse-bite-3mm-slot: VAL**, Panelization:mouse-bite-3mm-slot, F.Cu at (301.0, 34.5)
- added mouse-bite-3mm-slot: VAL**, Panelization:mouse-bite-3mm-slot, F.Cu at (301.0, 72.5)
- moved F1 11.5 mm to (291.5, 66.0)
- moved F13 11.0 mm to (35.0, 66.2)
Routing:
- net /Cell PCB/segment-n: track 17.5 -> 30.7 mm
- net /Cell PCB/segment-p: track 209.3 -> 221.9 mm
- net Net-(J13-Pin_1): track 14.7 -> 8.45 mm
- net Net-(J25-Pin_1): track 13.1 -> 8.28 mm
Other:
- outline, holes or cut-outs redrawn

Commit message: hopefully appease drc checker
Parts:
- moved NT1 0.62 mm to (267.4, 58.2)
Routing:
- net /Isolator/GLV-: track 48.6 -> 39.2 mm
- net GND: track 131.7 -> 126.4 mm
- net TEMP8: track 82.7 -> 81.2 mm
- net TEMP6: track 30.9 -> 30.0 mm
- net +3.3VA: track 33.8 -> 33.1 mm

Commit message: fix drc/erc errors
Parts:
- J29: footprint Connector_Dsub:DSUB-9_Female_Vertical_P2.77x2.84mm -> dsub:DSUB-9_Female_Vertical_P2.77x2.84mm
- J31: footprint Connector_Dsub:DSUB-15_Female_Vertical_P2.77x2.84mm -> dsub:DSUB-15_Female_Vertical_P2.77x2.84mm
Changed lines of the file:
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@@
         (effects (font (size 1 1) (thickness 0.15)))
     )
-    (fp_text user "*" (at -3.4163 -5.1689 -90) (layer "F.Fab")
+    (fp_text user "*" (at -3.4163 -5.1689 -90 unlocked) (layer "F.Fab")
         (effects (font (size 1 1) (thickness 0.15)))
     )
-    (fp_text user "${REFERENCE}" (at 0 0 -90 unlocked) (layer "F.Fab")
+    (fp_text user "*" (at -3.4163 -5.1689 -90) (layer "F.Fab")
         (effects (font (size 1 1) (thickness 0.15)))
     )
-    (fp_text user "*" (at -3.4163 -5.1689 -90 unlocked) (layer "F.Fab")
+    (fp_text user "${REFERENCE}" (at 0 0 -90 unlocked) (layer "F.Fab")
         (effects (font (size 1 1) (thickness 0.15)))
     )
@@
     )
   )
-  (footprint "Connector_Dsub:DSUB-9_Female_Vertical_P2.77x2.84mm" (layer "F.Cu")
+  (footprint "dsub:DSUB-9_Female_Vertical_P2.77x2.84mm" (layer "F.Cu")
     (at 309.66 44.45 180)
     (descr "9-pin D-Sub connector, straight/vertical, THT-mount, female, pitch 2.77x2.84mm, distance of mounting holes 25mm, see https://disti-assets.s3.amazonaws.com/tonar/files/datasheets/16730.pdf")
@@
     )
   )
-  (footprint "Connector_Dsub:DSUB-15_Female_Vertical_P2.77x2.84mm" (layer "F.Cu")
+  (footprint "dsub:DSUB-15_Female_Vertical_P2.77x2.84mm" (layer "F.Cu")
     (at 268.775 53.04)
     (descr "15-pin D-Sub connector, straight/vertical, THT-mount, female, pitch 2.77x2.84mm, distance of mounting holes 33.3mm, see https://disti-assets.s3.amazonaws.com/tonar/files/datasheets/16730.pdf")

Commit message: Kicad Update
Parts:
- removed C1, C10, C11, C12, C13, C14, C15, C16, C22, C3, C4, C5, C6, C7, C8, C9: 1u, Capacitor_SMD:C_0603_1608Metric
- removed C17: 4u7, Capacitor_SMD:C_0603_1608Metric
- removed C18, C19, C20, C21, C23: 100n, Capacitor_SMD:C_0603_1608Metric
- removed C24, C25: 30p, Capacitor_SMD:C_0603_1608Metric
- removed D10, D11, D12, D13, D14, D15, D17, D3, D5, D6, D7, D8, D9: RED 0603, LED_SMD:LED_0603_1608Metric
- removed F1, F10, F11, F12, F13, F2, F3, F4, F5, F6, F7, F8, F9: 2A 63VDC 1206, Fuse:Fuse_1206_3216Metric_Pad1.42x1.75mm_HandSolder
- removed FB1: 100R@100MHz, Resistor_SMD:R_0805_2012Metric
- removed G***: LOGO, art:stickbug
- removed G***: LOGO, art:pretzel
- removed J1, J10, J11, J12, J2, J3, J4, J6, J7, J8, J9: JST S2B-PH-SM4-TB, jst_conn:JST_PH_S2B-PH-SM4-TB_1x02-1MP_P2.00mm_Horizontal
- removed J13, J14, J15, J16, J17, J18, J19, J20, J21, J22, J23, J24, J25: Mounting Hole M5, MountingHole:MountingHole_5.3mm_M5_Pad_Via
- removed J26, J27: Pin Header 0.1" 01x04, Connector_PinHeader_2.54mm:PinHeader_1x04_P2.54mm_Vertical
- removed J28: TC2030, Connector:Tag-Connect_TC2030-IDC-NL_2x03_P1.27mm_Vertical
- removed J29: Norcomp 172-009-243R021, dsub:DSUB-9_Female_Vertical_P2.77x2.84mm
- removed JP1: SolderJumper_2_Bridged, Jumper:SolderJumper-2_P1.3mm_Bridged_RoundedPad1.0x1.5mm
- removed NT1: NetTie_2, NetTie:NetTie-2_SMD_Pad0.5mm
- removed R1, R11, R13, R15, R17, R19, R21, R23, R25, R27, R29, R31, R5, R7, R9: 10k 0.1%, Resistor_SMD:R_0603_1608Metric
- removed R10, R12, R14, R16, R18, R20, R22, R24, R26, R28, R30, R33, R6: 1k, Resistor_SMD:R_0603_1608Metric
- removed TH1, TH3, TH4: 10k NTC ERT-J1VR103J, Resistor_SMD:R_0603_1608Metric
- removed U1: STM32F103R8T6, Package_QFP:LQFP-64_10x10mm_P0.5mm
- removed Y1: 8MHz 20pF, Crystal:Crystal_SMD_5032-2Pin_5.0x3.2mm
- removed mouse-bite-3mm-slot (x3): VAL**, Panelization:mouse-bite-3mm-slot
- moved J5 50.0 mm to (327.5, 54.9)
- moved J31 41.6 mm to (309.5, 44.3), turned to 180 degrees
- moved J32 2.53 mm to (313.9, 25.5)
- moved J30 0.22 mm to (311.4, 81.5)
Connections:
- J31 pad 1: unconnected-(J31-Pad1) -> (no net)
- J31 pad 10: /Cell PCB/cell2-p -> (no net)
- J31 pad 11: /Cell PCB/cell4-p -> (no net)
- J31 pad 12: /Cell PCB/cell6-p -> (no net)
- J31 pad 13: /Cell PCB/cell8-p -> (no net)
- J31 pad 14: /Cell PCB/cell10-p -> (no net)
- J31 pad 15: /Cell PCB/segment-p -> (no net)
- J31 pad 2: /Cell PCB/cell1-p -> (no net)
- J31 pad 3: /Cell PCB/cell3-p -> (no net)
- J31 pad 4: /Cell PCB/cell5-p -> (no net)
- J31 pad 5: /Cell PCB/cell7-p -> (no net)
- J31 pad 6: /Cell PCB/cell9-p -> (no net)
- J31 pad 7: /Cell PCB/cell11-p -> (no net)
- J31 pad 8: unconnected-(J31-Pad8) -> (no net)
- J31 pad 9: /Cell PCB/segment-n -> (no net)
- J5 pad 1: TEMP0 -> (no net)
- J5 pad 2: GND -> (no net)
Routing:
- net /Cell PCB/segment-p: track 221.9 -> 0.00 mm
- net /Cell PCB/cell11-p: track 198.9 -> 0.00 mm
- net /Cell PCB/cell10-p: track 176.1 -> 0.00 mm
- net /Cell PCB/cell9-p: track 155.1 -> 0.00 mm
- net TEMP13: track 153.5 -> 0.00 mm, vias 2 -> 0
- net TEMP1: track 138.0 -> 0.00 mm, vias 2 -> 0
- net /Cell PCB/cell8-p: track 132.3 -> 0.00 mm
- net TEMP0: track 132.0 -> 0.00 mm, vias 2 -> 0
- net STAT1: track 130.7 -> 0.00 mm, vias 2 -> 0
- net TEMP11: track 130.3 -> 0.00 mm
- net TEMP10: track 129.0 -> 0.00 mm
- net GND: track 126.4 -> 0.00 mm, vias 39 -> 0
- net STAT11: track 124.5 -> 0.00 mm, vias 2 -> 0
- net TEMP12: track 124.3 -> 0.00 mm, vias 2 -> 0
- net STAT10: track 120.9 -> 0.00 mm, vias 2 -> 0
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- removed copper zone on In2.Cu, net +3.3VA
- removed copper zone on In2.Cu, net +3V3
- removed copper zone on In1.Cu, net GND
Other:
- board size 300.9 x 61.1 mm -> 30.3 x 61.3 mm
- board text removed: "+"
- board text removed: "+ 10 8 6 4 2 -"
- board text removed: "-"
- board text removed: "11 9 7 5 3 1"
- board text removed: "ALWAYS ENERGIZED"
- board text removed: "CANTX CANRX 3V3"
- board text removed: "CAUTION"
- board text removed: "Cell Tap & RTD interface"
- board text removed: "NOT ALWAYS ENERGIZED"
- board text removed: "NOT CAUTION"
- board text removed: "S1"
- board text removed: "S10"
- board text removed: "S11"
- board text removed: "S12"
- board text removed: "S2"
- board text removed: "S3"
- board text removed: "S4"
- board text removed: "S5"
- board text removed: "S6"
- board text removed: "S7"
- board text removed: "S9"
- board text removed: "THIS SIDE DOWN"
- board text removed: "if you are reading this text, this segment is assembled incorrectly."
- board text removed: "you just lost the game"
