File: cell-tap-connector-pcb.kicad_sch (KiCad schematic)
At the start: 0 parts

Commit message: more layout and memes
Other:
- sheet Isolater renamed Isolator
Changed lines of the file:
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@@
     (stroke (width 0.1524) (type solid))
     (fill (color 0 0 0 0.0000))
-    (property "Sheetname" "Isolater" (at 149.86 62.7884 0)
+    (property "Sheetname" "Isolator" (at 149.86 62.7884 0)
       (effects (font (size 1.27 1.27)) (justify left bottom))
     )
