File: thermistor_smd.kicad_sch (KiCad schematic)
At the start: 3 parts

Commit message: more layout and memes
Parts:
- C16: LibRef (none) -> CL10A105KA8NNNC; SKU (none) -> CL10A105KA8NNNC; Supplier (none) -> Digikey
- TH4: value 10k NTC -> 10k NTC ERT-J1VR103J; LibRef (none) -> ERT-J1VR103J; SKU (none) -> ERT-J1VR103J; Supplier (none) -> Digikey
Changed lines of the file:
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@@
+      (effects (font (size 1.27 1.27)) hide)
+    )
+    (property "LibRef" "" (at 157.48 91.44 0)
+      (effects (font (size 1.27 1.27)) hide)
+    )
+    (property "SKU" "" (at 157.48 91.44 0)
+      (effects (font (size 1.27 1.27)) hide)
+    )
+    (property "Supplier" "" (at 157.48 91.44 0)
       (effects (font (size 1.27 1.27)) hide)
     )
@@
       (effects (font (size 1.27 1.27)) (justify left))
     )
-    (property "Value" "10k NTC" (at 172.72 107.95 0)
+    (property "Value" "10k NTC ERT-J1VR103J" (at 172.72 107.95 0)
       (effects (font (size 1.27 1.27)) (justify left))
     )
@@
     )
     (property "Datasheet" "~" (at 168.91 106.68 0)
+      (effects (font (size 1.27 1.27)) hide)
+    )
+    (property "LibRef" "ERT-J1VR103J" (at 168.91 106.68 0)
+      (effects (font (size 1.27 1.27)) hide)
+    )
+    (property "SKU" "ERT-J1VR103J" (at 168.91 106.68 0)
+      (effects (font (size 1.27 1.27)) hide)
+    )
+    (property "Supplier" "Digikey" (at 168.91 106.68 0)
       (effects (font (size 1.27 1.27)) hide)
     )
@@
       (effects (font (size 1.27 1.27)) hide)
     )
+    (property "LibRef" "CL10A105KA8NNNC" (at 157.48 106.68 0)
+      (effects (font (size 1.27 1.27)) hide)
+    )
+    (property "SKU" "CL10A105KA8NNNC" (at 157.48 106.68 0)
+      (effects (font (size 1.27 1.27)) hide)
+    )
+    (property "Supplier" "Digikey" (at 157.48 106.68 0)
+      (effects (font (size 1.27 1.27)) hide)
+    )
+    (property "Description" "CAP CER 1UF 25V X5R 0603" (at 157.48 106.68 0)
+      (effects (font (size 1.27 1.27)) hide)
+    )

Commit message: Kicad Update
Parts:
- renumbered C16 to C1, R31 to R1, TH4 to TH1
